Commit message: modified urdf

File: content/assets/urdf/franka_description/franka_panda_no_gripper.urdf (robot description, URDF)
Before this commit: robot panda, 11 links, 10 joints
Links:
- added link panda_link8
- link panda_hand: geometry collision mesh filename=meshes/visual/hand_gripper.obj; visual mesh filename=meshes/visual/hand_gripper.stl
Joints:
- added joint panda_joint8: type fixed, parent panda_link7, child panda_link8, origin xyz=0 0 0.107 rpy=0 0 0, axis 0 0 0
- joint panda_hand_joint: origin xyz=0 0 0.107 rpy=0 0 -0.785398163397 -> xyz=0 0 0 rpy=0 0 -0.785398163397; parent panda_link7 -> panda_link8
